Commit message: namespaces look fine - issue with setting param server

File: src/virtualStingray_description/urdf/robot_simplified.urdf (robot description, URDF)
Before this commit: robot stingray, 5 links, 4 joints
Joints:
- joint R1_2nd_link_to_3rd_link: limit (none) -> lower=6.022 upper=0.262 effort=1000 velocity=10.0; type fixed -> revolute
- joint R1_3rd_link_to_4th_link: limit (none) -> lower=6.022 upper=0.262 effort=1000 velocity=10.0; type fixed -> revolute
- joint R1_4th_link_to_5th_link: limit (none) -> lower=6.022 upper=0.262 effort=1000 velocity=10.0; type fixed -> revolute
- joint R1_base_link_to_2nd_link: limit lower=-0.38 upper=0 effort=1000.0 velocity=0.5 -> lower=6.022 upper=0.262 effort=1000 velocity=10.0; type fixed -> revolute
